File: pcb/basalt-pcb.kicad_pcb (KiCad board)
At the start: 2 copper layers, 29 x 42 mm, 12 parts, among them J1 Conn_01x07_Pin, J2 Conn_01x07_Pin, J3 USB4215-03-A, J4 Conn_01x04_Pin, U1 DI78L3.3ZAB, U2 STM32C071F8Px

Commit message: Minor edits to pcb and titleblocks
Other:
- board text added: "Basalt Rev${REVISION}"
- board text removed: "Basalt Rev2"
Changed lines of the file:
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@@
 	)
 	(paper "A4")
+	(title_block
+		(title "MESA Basalt")
+		(date "2026-05-02")
+		(rev "2")
+		(company "OC ECE MESA")
+	)
 	(layers
 		(0 "F.Cu" signal)
@@
 		)
 	)
-	(gr_text "Basalt Rev2"
+	(gr_text "Basalt Rev${REVISION}"
 		(at 154.8 89.8 90)
 		(layer "B.SilkS")

Commit message: Fix mounting holes
Parts:
- added H1: MountingHole_Pad, MountingHole:MountingHole_2.2mm_M2_Pad, F.Cu at (138.0, 80.0)
- added H2: MountingHole_Pad, MountingHole:MountingHole_2.2mm_M2_Pad, F.Cu at (161.0, 80.0)
- added H3: MountingHole_Pad, MountingHole:MountingHole_2.2mm_M2_Pad, F.Cu at (138.0, 116.0)
- added H4: MountingHole_Pad, MountingHole:MountingHole_2.2mm_M2_Pad, F.Cu at (161.0, 116.0)
Other:
- outline, holes or cut-outs redrawn
